File: stuff/examples/counters/counters.kicad_sch (KiCad schematic)
At the start: 13 parts, among them U1 MAX7375AXR805, U2 74LS393, U3 74LS393, U4 74LS393, U5 74LS393, U6 74LS393, U7 74LS393, U8 74LS393, U9 74LS393

Commit message: reintroduce oscilloscope
Parts:
- removed U5, U6, U7, U8, U9: 74LS393, symbol 74xx:74LS393
- added U1: 74LS393, Package_DIP:DIP-14_W7.62mm, symbol 74xx:74LS393
- added unit 2 of U2
- added unit 2 of U3
- added unit 2 of U4
- Led1, Led2, Led3, Led4: footprint (none) -> LED_THT:LED_D5.0mm_Horizontal_O1.27mm_Z3.0mm_IRGrey
- OSC1: renamed from U1; footprint (none) -> Package_TO_SOT_SMD:SOT-323_SC-70
- U2, U3, U4: footprint (none) -> Package_DIP:DIP-14_W7.62mm
Connections:
- net at U2.1 (CP): now also U1.8 (Q3); no longer OSC1.2 (CLOCK)
- net at U3.1 (CP): now also U2.8 (Q3); no longer U2.6 (Q3)
- net at Led1.1 (IN): now also U4.11 (Q0)
- net at U4.6 (Q3): now also U4.13 (CP)
- net at U3.6 (Q3): now also U3.13 (CP); no longer U4.1 (CP)
- net at Led2.1 (IN): now also U4.10 (Q1)
- net at Led3.1 (IN): now also U4.9 (Q2)
- net at Led4.1 (IN): now also U4.8 (Q3)
- new net: U1.13 (CP), U1.6 (Q3)
- new net: OSC1.2 (CLOCK), U1.1 (CP)
- new net: U2.13 (CP), U2.6 (Q3)
- new net: U3.8 (Q3), U4.1 (CP)
Other:
- moved on the sheet: OSC1

Commit message: Oscillator   Enter frequency instead of period.   Hold target frequency more precise.   Show achieved frequency in desc. Readme
Parts:
- OSC1: SymPartParam (none) -> start
Changed lines of the file:
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@@
+      (effects (font (size 1.27 1.27)) hide)
+    )
+    (property "SymPartParam" "start" (at 107.95 39.37 0)
       (effects (font (size 1.27 1.27)) hide)
     )

Commit message: cleanup
Parts:
- OSC1: SymPartParam start -> (none)
Changed lines of the file:
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@@
-      (effects (font (size 1.27 1.27)) hide)
-    )
-    (property "SymPartParam" "start" (at 107.95 39.37 0)
       (effects (font (size 1.27 1.27)) hide)
     )
